Commit message: robot can be controlled w/ keyboard in gazebo

File: description/robot.urdf.xacro (robot description, xacro)
@@ -1,4 +1,5 @@
 <?xml version="1.0"?>
 <robot xmlns:xacro="http://www.ros.org/wiki/xacro" name="robot">
-    <xacro:include filename="robot_body.xacro" />
+  <xacro:include filename="robot_body.xacro" />
+  <xacro:include filename="robot_control.xacro" />
 </robot>

File: description/robot_body.xacro (robot description, xacro)
@@ -14,7 +14,13 @@
         <color rgba="1 1 0 1" />
     </material>
+    <material name="orange">
+        <color rgba="1 0.65 0 1" />
+    </material>
     <!-- BASE LINK -->
     <!-- let world origin at between centre of two wheels -->
     <link name="base_link">
+        <xacro:inertial_box mass="0.0001" x="0.0001" y="0.0001" z="0.0001">
+            <origin xyz="0 0 0" rpy="0 0 0" />
+        </xacro:inertial_box>
     </link>
     <!-- BODY -->
@@ -31,5 +37,5 @@
                 <box size="0.19 0.26 0.10" />
             </geometry>
-            <material name="white"/>
+            <material name="orange"/>
         </visual>
         <collision>
@@ -70,4 +76,9 @@
         </xacro:inertial_cylinder>
     </link>
+    <transmission name="left_wheel_trans">
+        <type>transmission_interface/SimpleTransmission</type>
+        <actuator name="left_wheel_motor"/>
+        <joint name="left_wheel_joint"/>
+    </transmission>
     <!-- RIGHT WHEEL -->
     <joint name="right_wheel_joint" type="continuous">
@@ -97,4 +108,9 @@
         </xacro:inertial_cylinder>
     </link>
+    <transmission name="right_wheel_trans">
+        <type>transmission_interface/SimpleTransmission</type>
+        <actuator name="right_wheel_motor"/>
+        <joint name="right_wheel_joint"/>
+    </transmission>
     <!-- CASTER WHEEL -->
     <joint name="caster_wheel_joint" type="fixed">

Commit message: ? gazebo sim works now ? rviz cant see laserscan

File: description/robot.urdf.xacro (robot description, xacro)
@@ -2,4 +2,7 @@
 <robot xmlns:xacro="http://www.ros.org/wiki/xacro" name="robot">
   <xacro:include filename="robot_body.xacro" />
-  <xacro:include filename="robot_control.xacro" />
+  <!-- <xacro:include filename="robot_control.xacro" /> -->
+  <xacro:include filename="lidar.xacro" />
+  <xacro:include filename="camera.xacro" />
+  <xacro:include filename="robot.gazebo" />
 </robot>

File: description/robot_body.xacro (robot description, xacro)
@@ -7,4 +7,7 @@
     <material name="black">
         <color rgba="0 0 0 1" />
+    </material>
+    <material name="gray">
+        <color rgba="0.5 0.5 0.5 1" />
     </material>
     <material name="red">
@@ -59,4 +62,6 @@
              ANTICLOCKWISE TO MOVE FORWARD -->
         <axis xyz="0 0 1"/>
+        <limit effort="50000" velocity="10"/>
+        <!-- <dynamics damping="1.0" friction="1.0"/> -->
     </joint>
     <link name="left_wheel">
@@ -76,9 +81,9 @@
         </xacro:inertial_cylinder>
     </link>
-    <transmission name="left_wheel_trans">
+    <!-- <transmission name="left_wheel_trans">
         <type>transmission_interface/SimpleTransmission</type>
         <actuator name="left_wheel_motor"/>
         <joint name="left_wheel_joint"/>
-    </transmission>
+    </transmission> -->
     <!-- RIGHT WHEEL -->
     <joint name="right_wheel_joint" type="continuous">
@@ -91,4 +96,6 @@
              ANTICLOCKWISE TO MOVE FORWARD -->
         <axis xyz="0 0 -1"/>
+        <limit effort="50000" velocity="10"/>
+        <!-- <dynamics damping="1.0" friction="1.0"/> -->
     </joint>
     <link name="right_wheel">
@@ -108,9 +115,9 @@
         </xacro:inertial_cylinder>
     </link>
-    <transmission name="right_wheel_trans">
+    <!-- <transmission name="right_wheel_trans">
         <type>transmission_interface/SimpleTransmission</type>
         <actuator name="right_wheel_motor"/>
         <joint name="right_wheel_joint"/>
-    </transmission>
+    </transmission> -->
     <!-- CASTER WHEEL -->
     <joint name="caster_wheel_joint" type="fixed">

Commit message: added ros2_control, may conflict w/ gazebo's plugins (currently commented out)

File: description/robot.urdf.xacro (robot description, xacro)
@@ -5,4 +5,7 @@
   <xacro:include filename="lidar.xacro" />
   <xacro:include filename="camera.xacro" />
+  <!-- for gazebo -->
   <xacro:include filename="robot.gazebo" />
+  <!-- for ros2_control: comment if use gz control -->
+  <xacro:include filename="ros2_control.xacro" />
 </robot>

File: description/robot_body.xacro (robot description, xacro)
@@ -74,5 +74,6 @@
         <collision>
             <geometry>
-                <cylinder radius="0.0335" length="0.027"/>
+                <!-- <cylinder radius="0.0335" length="0.027"/> -->
+                <sphere radius="0.0335" />
             </geometry>
         </collision>
@@ -108,5 +109,7 @@
         <collision>
             <geometry>
-                <cylinder radius="0.0335" length="0.027"/>
+                <!-- change geometry to sphere: reduce friction, make gazebo & rviz odom rotation more accurate -->
+                <!-- <cylinder radius="0.0335" length="0.027"/> -->
+                <sphere radius="0.0335" />
             </geometry>
         </collision>

Commit message: now can ctrl actual robot? haven't tested just commit so can copy to rpi

File: description/robot.urdf.xacro (robot description, xacro)
@@ -4,5 +4,5 @@
   <xacro:include filename="lidar.xacro" />
   <xacro:include filename="camera.xacro" />
-  <!-- gazebo sensors & physics  -->
+  <!-- gazebo sensor visuals & physics  -->
   <xacro:include filename="robot.gazebo" />
   <!-- Motor control: select one based on use_ros2_control argument -->

File: description/ros2_control.xacro (robot description, xacro)
@@ -1,7 +1,35 @@
 <?xml version="1.0"?>
 <robot xmlns:xacro="http://www.ros.org/wiki/xacro" name="robot">
-  <ros2_control name="GazeboSystem" type="system">
+  <!-- <ros2_control name="GazeboSystem" type="system">
     <hardware>
       <plugin>gz_ros2_control/GazeboSimSystem</plugin>
+    </hardware>
+    <joint name="left_wheel_joint">
+      <command_interface name="velocity">
+        <param name="min">-10</param>
+        <param name="max">10</param>
+      </command_interface>
+      <state_interface name="position"/>
+      <state_interface name="velocity"/>
+    </joint>
+    <joint name="right_wheel_joint">
+      <command_interface name="velocity">
+        <param name="min">-10</param>
+        <param name="max">10</param>
+      </command_interface>
+      <state_interface name="position"/>
+      <state_interface name="velocity"/>
+    </joint>
+  </ros2_control> -->
+  <ros2_control name="RealRobot" type="system">
+    <hardware>
+      <plugin>diffdrive_arduino/DiffDriveArduino</plugin>
+      <param name="left_wheel_name">left_wheel_joint</param>
+      <param name="right_wheel_name">right_wheel_joint</param>
+      <param name="loop_rate">30</param>
+      <param name="device">/dev/ttyUSB0</param>
+      <param name="baud_rate">115200</param>
+      <param name="timeout_ms">1000</param>
+      <param name="enc_counts_per_rev">3936</param>
     </hardware>
     <joint name="left_wheel_joint">
