Commit message: created URDF files

File: description/robot_body.xacro (robot description, xacro)
@@ -1,4 +1,5 @@
 <?xml version="1.0"?>
 <robot xmlns:xacro="http://www.ros.org/wiki/xacro">
+    <xacro:include filename="inertial_macros.xacro"/>
     <material name="white">
         <color rgba="1 1 1 1" />
@@ -36,4 +37,7 @@
             </geometry>
         </collision>
+        <xacro:inertial_box mass="0.5" x="0.3" y="0.3" z="0.15">
+            <origin xyz="0.15 0 0.075" rpy="0 0 0" />
+        </xacro:inertial_box>
     </link>
     <!-- LEFT WHEEL -->
@@ -60,4 +64,9 @@
             </geometry>
         </collision>
+        <xacro:inertial_cylinder mass="0.1" radius="0.05" length="0.04">
+            <origin xyz="0 0 0" rpy="0 0 0" />
+        </xacro:inertial_cylinder>
+            <origin xyz="0.15 0 0.075" rpy="0 0 0" />
+        </xacro:inertial_box>
     </link>
     <!-- RIGHT WHEEL -->
@@ -84,4 +93,7 @@
             </geometry>
         </collision>
+        <xacro:inertial_cylinder mass="0.1" radius="0.05" length="0.04">
+            <origin xyz="0 0 0" rpy="0 0 0" />
+        </xacro:inertial_cylinder>
     </link>
     <!-- CASTER WHEEL -->
@@ -103,4 +115,7 @@
             </geometry>
         </collision>
+        <xacro:inertial_sphere mass="0.1" radius="0.05">
+            <origin xyz="0 0 0" rpy="0 0 0" />
+        </xacro:inertial_cylinder>
     </link>
 </robot>

Commit message: edited urdf file to match actual robot

File: description/robot_body.xacro (robot description, xacro)
@@ -15,4 +15,5 @@
     </material>
     <!-- BASE LINK -->
+    <!-- let world origin at between centre of two wheels -->
     <link name="base_link">
     </link>
@@ -21,22 +22,23 @@
         <parent link="base_link" />
         <child link="body" />
-        <origin xyz="-0.1 0 0" />
+        <!-- joint at body's bottom rear-->
+        <origin xyz="-0.05 0 -0.025" />
     </joint>
     <link name="body">
         <visual>
-            <origin xyz="0.15 0 0.075" />
+            <origin xyz="0.095 0 0.05" />
             <geometry>
-                <box size="0.3 0.3 0.15" />
+                <box size="0.19 0.26 0.10" />
             </geometry>
             <material name="white"/>
         </visual>
         <collision>
-            <origin xyz="0.15 0 0.075" />
+            <origin xyz="0.095 0 0.05" />
             <geometry>
-                <box size="0.3 0.3 0.15" />
+                <box size="0.19 0.26 0.10" />
             </geometry>
         </collision>
-        <xacro:inertial_box mass="0.5" x="0.3" y="0.3" z="0.15">
-            <origin xyz="0.15 0 0.075" rpy="0 0 0" />
+        <xacro:inertial_box mass="1.2" x="0.19" y="0.26" z="0.1">
+            <origin xyz="0.095 0 0.05" rpy="0 0 0" />
         </xacro:inertial_box>
     </link>
@@ -47,5 +49,5 @@
         <!-- ROTATE Z-AXIS TO FACE OUTWARDS
              BY DEFAULT CYLINDER LENGTH PARALLEL TO Z-AXIS -->
-        <origin xyz="0 0.175 0" rpy="-${pi/2} 0 0"/>
+        <origin xyz="0 0.1435 0" rpy="-${pi/2} 0 0"/>
         <!-- WHEEL ROTATE AROUND Z-AXIS
              ANTICLOCKWISE TO MOVE FORWARD -->
@@ -55,5 +57,5 @@
         <visual>
             <geometry>
-                <cylinder radius="0.05" length="0.04"/>
+                <cylinder radius="0.0335" length="0.027"/>
             </geometry>
             <material name="black"/>
@@ -61,12 +63,10 @@
         <collision>
             <geometry>
-                <cylinder radius="0.05" length="0.04"/>
+                <cylinder radius="0.0335" length="0.027"/>
             </geometry>
         </collision>
-        <xacro:inertial_cylinder mass="0.1" radius="0.05" length="0.04">
+        <xacro:inertial_cylinder mass="0.05" radius="0.0335" length="0.027">
             <origin xyz="0 0 0" rpy="0 0 0" />
         </xacro:inertial_cylinder>
-            <origin xyz="0.15 0 0.075" rpy="0 0 0" />
-        </xacro:inertial_box>
     </link>
     <!-- RIGHT WHEEL -->
@@ -76,5 +76,5 @@
         <!-- ROTATE Z-AXIS TO FACE OUTWARDS
              BY DEFAULT CYLINDER LENGTH PARALLEL TO Z-AXIS -->
-        <origin xyz="0 -0.175 0" rpy="${pi/2} 0 0"/>
+        <origin xyz="0 -0.1435 0" rpy="${pi/2} 0 0"/>
         <!-- WHEEL ROTATE AROUND Z-AXIS
              ANTICLOCKWISE TO MOVE FORWARD -->
@@ -84,5 +84,5 @@
         <visual>
             <geometry>
-                <cylinder radius="0.05" length="0.04"/>
+                <cylinder radius="0.0335" length="0.027"/>
             </geometry>
             <material name="black"/>
@@ -90,8 +90,8 @@
         <collision>
             <geometry>
-                <cylinder radius="0.05" length="0.04"/>
+                <cylinder radius="0.0335" length="0.027"/>
             </geometry>
         </collision>
-        <xacro:inertial_cylinder mass="0.1" radius="0.05" length="0.04">
+        <xacro:inertial_cylinder mass="0.05" radius="0.0335" length="0.027">
             <origin xyz="0 0 0" rpy="0 0 0" />
         </xacro:inertial_cylinder>
@@ -101,10 +101,10 @@
         <parent link="body"/>
         <child link="caster_wheel"/>
-        <origin xyz="0.24 0 0"/>
+        <origin xyz="0.15 0 0"/>
     </joint>
     <link name="caster_wheel">
         <visual>
             <geometry>
-                <sphere radius="0.05"/>
+                <sphere radius="0.0085"/>
             </geometry>
             <material name="black"/>
@@ -112,10 +112,10 @@
         <collision>
             <geometry>
-                <sphere radius="0.05"/>
+                <sphere radius="0.0085"/>
             </geometry>
         </collision>
-        <xacro:inertial_sphere mass="0.1" radius="0.05">
+        <xacro:inertial_sphere mass="0.025" radius="0.0085">
             <origin xyz="0 0 0" rpy="0 0 0" />
-        </xacro:inertial_cylinder>
+        </xacro:inertial_sphere>
     </link>
 </robot>

Commit message: added slam stuff. can't load pre-saved map into rviz (localization)

File: description/robot_body.xacro (robot description, xacro)
@@ -26,4 +26,12 @@
             <origin xyz="0 0 0" rpy="0 0 0" />
         </xacro:inertial_box>
+    </link>
+    <!-- BASE_FOOTPRINT -->
+    <joint name="base_footprint_joint" type="fixed">
+        <parent link="base_link"/>
+        <child link="base_footprint"/>
+        <origin xyz="0 0 0" rpy="0 0 0"/>
+    </joint>
+    <link name="base_footprint">
     </link>
     <!-- BODY -->

File: description/ros2_control.xacro (robot description, xacro)
@@ -39,5 +39,5 @@
         <param name="right_wheel_name">right_wheel_joint</param>
         <param name="loop_rate">30</param>
-        <param name="device">/dev/ttyUSB0</param>
+        <param name="device">/dev/esp32</param>
         <param name="baud_rate">115200</param>
         <param name="timeout_ms">1000</param>
