Commit message: fix simulation  "camera" display in rviz (use temp_sim.launch.py & gz_bridge.yaml instead), tested later stuff (slam nav) also ok. Actual robot dk yet

File: description/camera.xacro (robot description, xacro)
@@ -4,5 +4,5 @@
     <parent link="body"/>
     <child link="camera_link"/>
-    <origin xyz="0.19 0 0.045" rpy="0 0 0"/>
+    <origin xyz="0.19 0 0.045" rpy="0 0.18 0"/> <!--tilt down cam by 0.18 rad-->
   </joint>
   <link name="camera_link">
@@ -16,8 +16,8 @@
   <joint name="camera_optical_joint" type="fixed">
     <parent link="camera_link"/>
-    <child link="camera_optical_link"/>
+    <child link="camera_link_optical"/>
     <origin xyz="0 0 0" rpy="${-pi/2} 0 ${-pi/2}"/>
   </joint>
-  <link name="camera_optical_link">
+  <link name="camera_link_optical">
   </link>
 </robot>
